Commit message: Adding Lidar to URDF

File: description/robot.urdf.xacro (robot description, xacro)
@@ -2,3 +2,4 @@
 <robot xmlns:xacro="http://www.ros.org/wiki/xacro"  name="agv">
     <xacro:include filename="robot_core.xacro"/>
+    <xacro:include filename="lidar.xacro"/>
 </robot>

File: description/robot_core.xacro (robot description, xacro)
@@ -40,5 +40,4 @@
             <geometry>
                 <box size="${chassis_length} ${chassis_width} ${chassis_base_height}"/>
-                <!-- <mesh filename="file://home/ros/ros/agv_ws/src/agv_ros/meshes/agv_body.stl"/> -->
             </geometry>
             <material name="white"/>
@@ -48,5 +47,4 @@
             <geometry>
                 <box size="${chassis_length} ${chassis_width} ${chassis_base_height}"/>
-                <!-- <mesh filename="file://home/ros/ros/agv_ws/src/agv_ros/meshes/agv_body.stl"/> -->
             </geometry>
         </collision>
@@ -69,5 +67,4 @@
             <geometry>
                 <box size="${chassis_mid_length} ${chassis_width} ${chassis_mid_height}"/>
-                <!-- <mesh filename="file://home/ros/ros/agv_ws/src/agv_ros/meshes/agv_body.stl"/> -->
             </geometry>
             <material name="orange"/>
@@ -77,5 +74,4 @@
             <geometry>
                 <box size="${chassis_mid_length} ${chassis_width} ${chassis_mid_height}"/>
-                <!-- <mesh filename="file://home/ros/ros/agv_ws/src/agv_ros/meshes/agv_body.stl"/> -->
             </geometry>
         </collision>
@@ -85,5 +81,5 @@
     </link>
     <gazebo reference="mid_chassis">
-        <material>Gazebo/White</material>
+        <material>Gazebo/Orange</material>
     </gazebo>
     <!-- UPPER CHASSIS LINK -->
@@ -98,7 +94,6 @@
             <geometry>
                 <box size="${chassis_length} ${chassis_width} ${chassis_upper_height}"/>
-                <!-- <mesh filename="file://home/ros/ros/agv_ws/src/agv_ros/meshes/agv_body.stl"/> -->
-            </geometry>
-            <material name="white"/>
+            </geometry>
+            <material name="orange"/>
         </visual>
         <collision>
@@ -106,5 +101,4 @@
             <geometry>
                 <box size="${chassis_length} ${chassis_width} ${chassis_upper_height}"/>
-                <!-- <mesh filename="file://home/ros/ros/agv_ws/src/agv_ros/meshes/agv_body.stl"/> -->
             </geometry>
         </collision>
@@ -114,5 +108,5 @@
     </link>
     <gazebo reference="upper_chassis">
-        <material>Gazebo/White</material>
+        <material>Gazebo/Orange</material>
     </gazebo>
     <!-- LEFT WHEEL LINK -->
