Commit message: Changing Robot URDF

File: description/gazebo_control.xacro (robot description, xacro)
@@ -9,6 +9,6 @@
             <wheel_diameter>0.154</wheel_diameter>
             <!-- Limits -->
-            <max_wheel_torque>500</max_wheel_torque>
-            <max_wheel_acceleration>20.0</max_wheel_acceleration>
+            <max_wheel_torque>200</max_wheel_torque>
+            <max_wheel_acceleration>10.0</max_wheel_acceleration>
             <!-- Output -->
             <odometry_frame>odom</odometry_frame>

File: description/robot_core.xacro (robot description, xacro)
@@ -26,5 +26,5 @@
     <xacro:property name="caster_wheel_f_offset_x" value="0.560"/>
     <xacro:property name="caster_wheel_offset_y" value="0.20"/>
-    <xacro:property name="caster_wheel_offset_z" value="${wheel_offset_z - wheel_radius + caster_wheel_radius}"/>
+    <xacro:property name="caster_wheel_offset_z" value="${wheel_offset_z - wheel_radius + caster_wheel_radius + 0.0005}"/>
     <!-- BASE LINK -->
     <link name="base_link"></link>
@@ -186,6 +186,6 @@
     <gazebo reference="caster_wheel_br">
         <material>Gazebo/Black</material>
-        <mu1 value="0.001"/>
-        <mu2 value="0.001"/>
+        <mu1 value="0.005"/>
+        <mu2 value="0.005"/>
     </gazebo>
     <!-- CASTER WHEEL LINK BL-->
@@ -213,6 +213,6 @@
     <gazebo reference="caster_wheel_bl">
         <material>Gazebo/Black</material>
-        <mu1 value="0.001"/>
-        <mu2 value="0.001"/>
+        <mu1 value="0.005"/>
+        <mu2 value="0.005"/>
     </gazebo>
     <!-- CASTER WHEEL LINK FR-->
@@ -240,6 +240,6 @@
     <gazebo reference="caster_wheel_fr">
         <material>Gazebo/Black</material>
-        <mu1 value="0.001"/>
-        <mu2 value="0.001"/>
+        <mu1 value="0.004"/>
+        <mu2 value="0.004"/>
     </gazebo>
     <!-- CASTER WHEEL LINK FL-->
@@ -267,6 +267,6 @@
     <gazebo reference="caster_wheel_fl">
         <material>Gazebo/Black</material>
-        <mu1 value="0.001"/>
-        <mu2 value="0.001"/>
+        <mu1 value="0.004"/>
+        <mu2 value="0.004"/>
     </gazebo>
 </robot>
