Commit message: Creating Launch File

File: description/lidar.xacro (robot description, xacro)
@@ -42,5 +42,5 @@
         <parent link="lidar_chassis"/>
         <child link="laser_frame"/>
-        <origin xyz="0 0 ${lidar_chassis_height}" rpy="0 0 0"/>
+        <origin xyz="0 0 ${lidar_chassis_height + lidar_thickness/2}" rpy="0 0 0"/>
     </joint>
     <link name="laser_frame">
@@ -83,5 +83,5 @@
                 </scan>
                 <range>
-                    <min>0.3</min>
+                    <min>0.1</min>
                     <max>12</max>
                 </range>

File: description/robot.urdf.xacro (robot description, xacro)
@@ -3,3 +3,4 @@
     <xacro:include filename="robot_core.xacro"/>
     <xacro:include filename="lidar.xacro"/>
+    <xacro:include filename="gazebo_control.xacro"/>
 </robot>

Commit message: Adding SLAM

File: description/lidar.xacro (robot description, xacro)
@@ -42,5 +42,5 @@
         <parent link="lidar_chassis"/>
         <child link="laser_frame"/>
-        <origin xyz="0 0 ${lidar_chassis_height + lidar_thickness/2}" rpy="0 0 0"/>
+        <origin xyz="0 0 ${lidar_chassis_height + lidar_thickness/2}" rpy="0 0 ${pi}"/>
     </joint>
     <link name="laser_frame">

File: description/ros2_control.xacro (robot description, xacro)
@@ -11,5 +11,5 @@
                 <param name="baud_rate">57600</param>
                 <param name="timeout">1000</param>
-                <param name="enc_counts_per_rev">237416</param>
+                <param name="enc_counts_per_rev">2374</param>
             </hardware>
             <joint name="left_wheel_joint">

Commit message: Change Lidar Coord

File: description/lidar.xacro (robot description, xacro)
@@ -15,5 +15,5 @@
         <parent link="chassis"/>
         <child link="lidar_chassis"/>
-        <origin xyz="${lidar_chassis_offset_x - lidar_chassis_length/2} 0 ${lidar_chassis_offset_z}"/>
+        <origin xyz="${lidar_chassis_offset_x - lidar_chassis_length/2} 0 ${lidar_chassis_offset_z}" rpy="0 0 ${pi}"/>
     </joint>
     <link name="lidar_chassis">
@@ -42,5 +42,5 @@
         <parent link="lidar_chassis"/>
         <child link="laser_frame"/>
-        <origin xyz="0 0 ${lidar_chassis_height + lidar_thickness/2}" rpy="0 0 ${pi}"/>
+        <origin xyz="0 0 ${lidar_chassis_height + lidar_thickness/2}" rpy="0 0 0"/>
     </joint>
     <link name="laser_frame">
@@ -78,6 +78,6 @@
                     <horizontal>
                         <samples>360</samples>
-                        <min_angle>-3.14</min_angle>
-                        <max_angle>3.14</max_angle>
+                        <min_angle>-1.57</min_angle>
+                        <max_angle>1.57</max_angle>
                     </horizontal>
                 </scan>
