Commit message: Adding Robot URDF

File: description/robot_core.xacro (robot description, xacro)
@@ -1,3 +1,212 @@
 <?xml version="1.0"?>
 <robot xmlns:xacro="http://www.ros.org/wiki/xacro">
+    <!-- INCLUDE SUPPORTING XACRO -->
+    <xacro:include filename="color.xacro"/>
+    <xacro:include filename="inertial_macros.xacro"/>
+    <!-- DEFINE ROBOT PROPERTIES -->
+    <xacro:property name="chassis_length" value="0.650"/>
+    <xacro:property name="chassis_width" value="0.500"/>
+    <xacro:property name="chassis_height" value="0.360"/>
+    <xacro:property name="chassis_mass" value="70.0"/>
+    <xacro:property name="wheel_radius" value="0.077"/>
+    <xacro:property name="wheel_thickness" value="0.04"/>
+    <xacro:property name="wheel_mass" value="0.5"/>
+    <xacro:property name="wheel_offset_x" value="0.325"/>
+    <xacro:property name="wheel_offset_y" value="0.21"/>
+    <xacro:property name="wheel_offset_z" value="0.05"/>
+    <xacro:property name="caster_wheel_radius" value="0.025"/>
+    <xacro:property name="caster_wheel_mass" value="0.1"/>
+    <xacro:property name="caster_wheel_f_offset_x" value="0.122"/>
+    <xacro:property name="caster_wheel_b_offset_x" value="0.580"/>
+    <xacro:property name="caster_wheel_offset_y" value="0.20"/>
+    <xacro:property name="caster_wheel_offset_z" value="${wheel_offset_z - wheel_radius + caster_wheel_radius}"/>
+    <!-- BASE LINK -->
+    <link name="base_link"></link>
+    <!-- CHASSIS LINK -->
+    <joint name="chassis_joint" type="fixed">
+        <parent link="base_link"/>
+        <child link="chassis"/>
+        <origin xyz="${-wheel_offset_x} 0 ${-wheel_offset_z}"/>
+    </joint>
+    <link name="chassis">
+        <visual>
+            <origin xyz="${chassis_length/2} 0 ${chassis_height/2}"/>
+            <geometry>
+                <box size="${chassis_length} ${chassis_width} ${chassis_height}"/>
+            </geometry>
+            <material name="white"/>
+        </visual>
+        <collision>
+            <origin xyz="${chassis_length/2} 0 ${chassis_height/2}"/>
+            <geometry>
+                <box size="${chassis_length} ${chassis_width} ${chassis_height}"/>
+            </geometry>
+        </collision>
+        <xacro:inertial_box mass="${chassis_mass}" x="${chassis_length}" y="${chassis_width}" z="${chassis_height}">
+            <origin xyz="${chassis_length/2} 0 ${chassis_height/2}" rpy="0 0 0"/>
+        </xacro:inertial_box>
+    </link>
+    <gazebo reference="chassis">
+        <material>Gazebo/White</material>
+    </gazebo>
+    <!-- LEFT WHEEL LINK -->
+    <joint name="left_wheel_joint" type="continuous">
+        <parent link="base_link"/>
+        <child link="left_wheel"/>
+        <origin xyz="0 ${wheel_offset_y} 0" rpy="-${pi/2} 0 0" />
+        <axis xyz="0 0 1"/>
+    </joint>
+    <link name="left_wheel">
+        <visual>
+            <geometry>
+                <cylinder radius="${wheel_radius}" length="${wheel_thickness}"/>
+            </geometry>
+            <material name="blue"/>
+        </visual>
+        <collision>
+            <geometry>
+                <sphere radius="${wheel_radius}"/>
+            </geometry>
+        </collision>
+        <xacro:inertial_cylinder mass="${wheel_mass}" length="${wheel_thickness}" radius="${wheel_radius}">
+            <origin xyz="0 0 0" rpy="0 0 0"/>
+        </xacro:inertial_cylinder>
+    </link>
+    <gazebo reference="left_wheel">
+        <material>Gazebo/Blue</material>
+    </gazebo>
+    <!-- RIGHT WHEEL LINK -->
+    <joint name="right_wheel_joint" type="continuous">
+        <parent link="base_link"/>
+        <child link="right_wheel"/>
+        <origin xyz="0 ${-wheel_offset_y} 0" rpy="${pi/2} 0 0" />
+        <axis xyz="0 0 -1"/>
+    </joint>
+    <link name="right_wheel">
+        <visual>
+            <geometry>
+                <cylinder radius="${wheel_radius}" length="${wheel_thickness}"/>
+            </geometry>
+            <material name="blue"/>
+        </visual>
+        <collision>
+            <geometry>
+                <sphere radius="${wheel_radius}"/>
+            </geometry>
+        </collision>
+        <xacro:inertial_cylinder mass="${wheel_mass}" length="${wheel_thickness}" radius="${wheel_radius}">
+            <origin xyz="0 0 0" rpy="0 0 0"/>
+        </xacro:inertial_cylinder>
+    </link>
+    <gazebo reference="right_wheel">
+        <material>Gazebo/Blue</material>
+    </gazebo>
+    <!-- CASTER WHEEL LINK FR-->
+    <joint name="caster_wheel_fr_joint" type="fixed">
+        <parent link="chassis"/>
+        <child link="caster_wheel_fr"/>
+        <origin xyz="${caster_wheel_f_offset_x} ${-caster_wheel_offset_y} ${caster_wheel_offset_z}"/>
+    </joint>
+    <link name="caster_wheel_fr">
+        <visual>
+            <geometry>
+                <sphere radius="${caster_wheel_radius}"/>
+            </geometry>
+            <material name="black"/>
+        </visual>
+        <collision>
+            <geometry>
+                <sphere radius="${caster_wheel_radius}"/>
+            </geometry>
+        </collision>
+        <xacro:inertial_sphere mass="${caster_wheel_mass}" radius="${caster_wheel_radius}">
+            <origin xyz="0 0 0" rpy="0 0 0"/>
+        </xacro:inertial_sphere>
+    </link>
+    <gazebo reference="caster_wheel_fr">
+        <material>Gazebo/Black</material>
+        <mu1 value="0.001"/>
+        <mu2 value="0.001"/>
+    </gazebo>
+    <!-- CASTER WHEEL LINK FL-->
+    <joint name="caster_wheel_fl_joint" type="fixed">
+        <parent link="chassis"/>
+        <child link="caster_wheel_fl"/>
+        <origin xyz="${caster_wheel_f_offset_x} ${caster_wheel_offset_y} ${caster_wheel_offset_z}"/>
+    </joint>
+    <link name="caster_wheel_fl">
+        <visual>
+            <geometry>
+                <sphere radius="${caster_wheel_radius}"/>
+            </geometry>
+            <material name="black"/>
+        </visual>
+        <collision>
+            <geometry>
+                <sphere radius="${caster_wheel_radius}"/>
+            </geometry>
+        </collision>
+        <xacro:inertial_sphere mass="${caster_wheel_mass}" radius="${caster_wheel_radius}">
+            <origin xyz="0 0 0" rpy="0 0 0"/>
+        </xacro:inertial_sphere>
+    </link>
+    <gazebo reference="caster_wheel_fl">
+        <material>Gazebo/Black</material>
+        <mu1 value="0.001"/>
+        <mu2 value="0.001"/>
+    </gazebo>
+    <!-- CASTER WHEEL LINK BR-->
+    <joint name="caster_wheel_br_joint" type="fixed">
+        <parent link="chassis"/>
+        <child link="caster_wheel_br"/>
+        <origin xyz="${caster_wheel_b_offset_x} ${-caster_wheel_offset_y} ${caster_wheel_offset_z}"/>
+    </joint>
+    <link name="caster_wheel_br">
+        <visual>
+            <geometry>
+                <sphere radius="${caster_wheel_radius}"/>
+            </geometry>
+            <material name="black"/>
+        </visual>
+        <collision>
+            <geometry>
+                <sphere radius="${caster_wheel_radius}"/>
+            </geometry>
+        </collision>
+        <xacro:inertial_sphere mass="${caster_wheel_mass}" radius="${caster_wheel_radius}">
+            <origin xyz="0 0 0" rpy="0 0 0"/>
+        </xacro:inertial_sphere>
+    </link>
+    <gazebo reference="caster_wheel_br">
+        <material>Gazebo/Black</material>
+        <mu1 value="0.001"/>
+        <mu2 value="0.001"/>
+    </gazebo>
+    <!-- CASTER WHEEL LINK BL-->
+    <joint name="caster_wheel_bl_joint" type="fixed">
+        <parent link="chassis"/>
+        <child link="caster_wheel_bl"/>
+        <origin xyz="${caster_wheel_b_offset_x} ${caster_wheel_offset_y} ${caster_wheel_offset_z}"/>
+    </joint>
+    <link name="caster_wheel_bl">
+        <visual>
+            <geometry>
+                <sphere radius="${caster_wheel_radius}"/>
+            </geometry>
+            <material name="black"/>
+        </visual>
+        <collision>
+            <geometry>
+                <sphere radius="${caster_wheel_radius}"/>
+            </geometry>
+        </collision>
+        <xacro:inertial_sphere mass="${caster_wheel_mass}" radius="${caster_wheel_radius}">
+            <origin xyz="0 0 0" rpy="0 0 0"/>
+        </xacro:inertial_sphere>
+    </link>
+    <gazebo reference="caster_wheel_bl">
+        <material>Gazebo/Black</material>
+        <mu1 value="0.001"/>
+        <mu2 value="0.001"/>
+    </gazebo>
 </robot>

Commit message: Minor Changes URDF

File: description/robot_core.xacro (robot description, xacro)
@@ -17,6 +17,6 @@
     <xacro:property name="caster_wheel_radius" value="0.025"/>
     <xacro:property name="caster_wheel_mass" value="0.1"/>
-    <xacro:property name="caster_wheel_f_offset_x" value="0.122"/>
-    <xacro:property name="caster_wheel_b_offset_x" value="0.580"/>
+    <xacro:property name="caster_wheel_b_offset_x" value="0.122"/>
+    <xacro:property name="caster_wheel_f_offset_x" value="0.580"/>
     <xacro:property name="caster_wheel_offset_y" value="0.20"/>
     <xacro:property name="caster_wheel_offset_z" value="${wheel_offset_z - wheel_radius + caster_wheel_radius}"/>
@@ -33,5 +33,6 @@
             <origin xyz="${chassis_length/2} 0 ${chassis_height/2}"/>
             <geometry>
-                <box size="${chassis_length} ${chassis_width} ${chassis_height}"/>
+                <!-- <box size="${chassis_length} ${chassis_width} ${chassis_height}"/> -->
+                <mesh filename="package://$(find agv_ros)/meshes/AGV-Body-v2.stl"/>
             </geometry>
             <material name="white"/>
@@ -40,5 +41,6 @@
             <origin xyz="${chassis_length/2} 0 ${chassis_height/2}"/>
             <geometry>
-                <box size="${chassis_length} ${chassis_width} ${chassis_height}"/>
+                <!-- <box size="${chassis_length} ${chassis_width} ${chassis_height}"/> -->
+                <mesh filename="package://$(find agv_ros)/meshes/AGV-Body-v2.stl"/>
             </geometry>
         </collision>
@@ -102,4 +104,58 @@
         <material>Gazebo/Blue</material>
     </gazebo>
+    <!-- CASTER WHEEL LINK BR-->
+    <joint name="caster_wheel_br_joint" type="fixed">
+        <parent link="chassis"/>
+        <child link="caster_wheel_br"/>
+        <origin xyz="${caster_wheel_b_offset_x} ${-caster_wheel_offset_y} ${caster_wheel_offset_z}"/>
+    </joint>
+    <link name="caster_wheel_br">
+        <visual>
+            <geometry>
+                <sphere radius="${caster_wheel_radius}"/>
+            </geometry>
+            <material name="black"/>
+        </visual>
+        <collision>
+            <geometry>
+                <sphere radius="${caster_wheel_radius}"/>
+            </geometry>
+        </collision>
+        <xacro:inertial_sphere mass="${caster_wheel_mass}" radius="${caster_wheel_radius}">
+            <origin xyz="0 0 0" rpy="0 0 0"/>
+        </xacro:inertial_sphere>
+    </link>
+    <gazebo reference="caster_wheel_br">
+        <material>Gazebo/Black</material>
+        <mu1 value="0.001"/>
+        <mu2 value="0.001"/>
+    </gazebo>
+    <!-- CASTER WHEEL LINK BL-->
+    <joint name="caster_wheel_bl_joint" type="fixed">
+        <parent link="chassis"/>
+        <child link="caster_wheel_bl"/>
+        <origin xyz="${caster_wheel_b_offset_x} ${caster_wheel_offset_y} ${caster_wheel_offset_z}"/>
+    </joint>
+    <link name="caster_wheel_bl">
+        <visual>
+            <geometry>
+                <sphere radius="${caster_wheel_radius}"/>
+            </geometry>
+            <material name="black"/>
+        </visual>
+        <collision>
+            <geometry>
+                <sphere radius="${caster_wheel_radius}"/>
+            </geometry>
+        </collision>
+        <xacro:inertial_sphere mass="${caster_wheel_mass}" radius="${caster_wheel_radius}">
+            <origin xyz="0 0 0" rpy="0 0 0"/>
+        </xacro:inertial_sphere>
+    </link>
+    <gazebo reference="caster_wheel_bl">
+        <material>Gazebo/Black</material>
+        <mu1 value="0.001"/>
+        <mu2 value="0.001"/>
+    </gazebo>
     <!-- CASTER WHEEL LINK FR-->
     <joint name="caster_wheel_fr_joint" type="fixed">
@@ -156,57 +212,3 @@
         <mu2 value="0.001"/>
     </gazebo>
-    <!-- CASTER WHEEL LINK BR-->
-    <joint name="caster_wheel_br_joint" type="fixed">
-        <parent link="chassis"/>
-        <child link="caster_wheel_br"/>
-        <origin xyz="${caster_wheel_b_offset_x} ${-caster_wheel_offset_y} ${caster_wheel_offset_z}"/>
-    </joint>
-    <link name="caster_wheel_br">
-        <visual>
-            <geometry>
-                <sphere radius="${caster_wheel_radius}"/>
-            </geometry>
-            <material name="black"/>
-        </visual>
-        <collision>
-            <geometry>
-                <sphere radius="${caster_wheel_radius}"/>
-            </geometry>
-        </collision>
-        <xacro:inertial_sphere mass="${caster_wheel_mass}" radius="${caster_wheel_radius}">
-            <origin xyz="0 0 0" rpy="0 0 0"/>
-        </xacro:inertial_sphere>
-    </link>
-    <gazebo reference="caster_wheel_br">
-        <material>Gazebo/Black</material>
-        <mu1 value="0.001"/>
-        <mu2 value="0.001"/>
-    </gazebo>
-    <!-- CASTER WHEEL LINK BL-->
-    <joint name="caster_wheel_bl_joint" type="fixed">
-        <parent link="chassis"/>
-        <child link="caster_wheel_bl"/>
-        <origin xyz="${caster_wheel_b_offset_x} ${caster_wheel_offset_y} ${caster_wheel_offset_z}"/>
-    </joint>
-    <link name="caster_wheel_bl">
-        <visual>
-            <geometry>
-                <sphere radius="${caster_wheel_radius}"/>
-            </geometry>
-            <material name="black"/>
-        </visual>
-        <collision>
-            <geometry>
-                <sphere radius="${caster_wheel_radius}"/>
-            </geometry>
-        </collision>
-        <xacro:inertial_sphere mass="${caster_wheel_mass}" radius="${caster_wheel_radius}">
-            <origin xyz="0 0 0" rpy="0 0 0"/>
-        </xacro:inertial_sphere>
-    </link>
-    <gazebo reference="caster_wheel_bl">
-        <material>Gazebo/Black</material>
-        <mu1 value="0.001"/>
-        <mu2 value="0.001"/>
-    </gazebo>
 </robot>

Commit message: Tweaking Robot URDF

File: description/robot_core.xacro (robot description, xacro)
@@ -7,6 +7,12 @@
     <xacro:property name="chassis_length" value="0.650"/>
     <xacro:property name="chassis_width" value="0.500"/>
-    <xacro:property name="chassis_height" value="0.360"/>
-    <xacro:property name="chassis_mass" value="70.0"/>
+    <xacro:property name="chassis_height" value="0.320"/>
+    <xacro:property name="chassis_base_height" value="0.052"/>
+    <xacro:property name="chassis_base_mass" value="28.0"/>
+    <xacro:property name="chassis_mid_length" value="0.530"/>
+    <xacro:property name="chassis_mid_height" value="0.150"/>
+    <xacro:property name="chassis_mid_mass" value="28.0"/>
+    <xacro:property name="chassis_upper_height" value="0.118"/>
+    <xacro:property name="chassis_upper_mass" value="28.0"/>
     <xacro:property name="wheel_radius" value="0.077"/>
     <xacro:property name="wheel_thickness" value="0.04"/>
@@ -17,11 +23,11 @@
     <xacro:property name="caster_wheel_radius" value="0.025"/>
     <xacro:property name="caster_wheel_mass" value="0.1"/>
-    <xacro:property name="caster_wheel_b_offset_x" value="0.122"/>
-    <xacro:property name="caster_wheel_f_offset_x" value="0.580"/>
+    <xacro:property name="caster_wheel_b_offset_x" value="0.095"/>
+    <xacro:property name="caster_wheel_f_offset_x" value="0.560"/>
     <xacro:property name="caster_wheel_offset_y" value="0.20"/>
     <xacro:property name="caster_wheel_offset_z" value="${wheel_offset_z - wheel_radius + caster_wheel_radius}"/>
     <!-- BASE LINK -->
     <link name="base_link"></link>
-    <!-- CHASSIS LINK -->
+    <!-- BASE CHASSIS LINK -->
     <joint name="chassis_joint" type="fixed">
         <parent link="base_link"/>
@@ -31,23 +37,81 @@
     <link name="chassis">
         <visual>
-            <origin xyz="${chassis_length/2} 0 ${chassis_height/2}"/>
-            <geometry>
-                <!-- <box size="${chassis_length} ${chassis_width} ${chassis_height}"/> -->
-                <mesh filename="package://$(find agv_ros)/meshes/AGV-Body-v2.stl"/>
+            <origin xyz="${chassis_length/2} 0 ${chassis_base_height/2}"/>
+            <geometry>
+                <box size="${chassis_length} ${chassis_width} ${chassis_base_height}"/>
+                <!-- <mesh filename="file://home/ros/ros/agv_ws/src/agv_ros/meshes/agv_body.stl"/> -->
             </geometry>
             <material name="white"/>
         </visual>
         <collision>
-            <origin xyz="${chassis_length/2} 0 ${chassis_height/2}"/>
-            <geometry>
-                <!-- <box size="${chassis_length} ${chassis_width} ${chassis_height}"/> -->
-                <mesh filename="package://$(find agv_ros)/meshes/AGV-Body-v2.stl"/>
-            </geometry>
-        </collision>
-        <xacro:inertial_box mass="${chassis_mass}" x="${chassis_length}" y="${chassis_width}" z="${chassis_height}">
-            <origin xyz="${chassis_length/2} 0 ${chassis_height/2}" rpy="0 0 0"/>
+            <origin xyz="${chassis_length/2} 0 ${chassis_base_height/2}"/>
+            <geometry>
+                <box size="${chassis_length} ${chassis_width} ${chassis_base_height}"/>
+                <!-- <mesh filename="file://home/ros/ros/agv_ws/src/agv_ros/meshes/agv_body.stl"/> -->
+            </geometry>
+        </collision>
+        <xacro:inertial_box mass="${chassis_base_mass}" x="${chassis_length}" y="${chassis_width}" z="${chassis_base_height}">
+            <origin xyz="${chassis_length/2} 0 ${chassis_base_height/2}" rpy="0 0 0"/>
         </xacro:inertial_box>
     </link>
     <gazebo reference="chassis">
+        <material>Gazebo/White</material>
+    </gazebo>
+    <!-- MID CHASSIS LINK -->
+    <joint name="mid_chassis_joint" type="fixed">
+        <parent link="base_link"/>
+        <child link="mid_chassis"/>
+        <origin xyz="${-wheel_offset_x} 0 ${-wheel_offset_z}"/>
+    </joint>
+    <link name="mid_chassis">
+        <visual>
+            <origin xyz="${chassis_mid_length/2} 0 ${chassis_mid_height/2 + chassis_base_height}"/>
+            <geometry>
+                <box size="${chassis_mid_length} ${chassis_width} ${chassis_mid_height}"/>
+                <!-- <mesh filename="file://home/ros/ros/agv_ws/src/agv_ros/meshes/agv_body.stl"/> -->
+            </geometry>
+            <material name="orange"/>
+        </visual>
+        <collision>
+            <origin xyz="${chassis_mid_length/2} 0 ${chassis_mid_height/2 + chassis_base_height}"/>
+            <geometry>
+                <box size="${chassis_mid_length} ${chassis_width} ${chassis_mid_height}"/>
+                <!-- <mesh filename="file://home/ros/ros/agv_ws/src/agv_ros/meshes/agv_body.stl"/> -->
+            </geometry>
+        </collision>
+        <xacro:inertial_box mass="${chassis_mid_mass}" x="${chassis_mid_length}" y="${chassis_width}" z="${chassis_mid_height}">
+            <origin xyz="${chassis_mid_length/2} 0 ${chassis_mid_height/2 + chassis_base_height}" rpy="0 0 0"/>
+        </xacro:inertial_box>
+    </link>
+    <gazebo reference="mid_chassis">
+        <material>Gazebo/White</material>
+    </gazebo>
+    <!-- UPPER CHASSIS LINK -->
+    <joint name="upper_chassis_joint" type="fixed">
+        <parent link="base_link"/>
+        <child link="upper_chassis"/>
+        <origin xyz="${-wheel_offset_x} 0 ${-wheel_offset_z}"/>
+    </joint>
+    <link name="upper_chassis">
+        <visual>
+            <origin xyz="${chassis_length/2} 0 ${chassis_upper_height/2 + chassis_base_height + chassis_mid_height}"/>
+            <geometry>
+                <box size="${chassis_length} ${chassis_width} ${chassis_upper_height}"/>
+                <!-- <mesh filename="file://home/ros/ros/agv_ws/src/agv_ros/meshes/agv_body.stl"/> -->
+            </geometry>
+            <material name="white"/>
+        </visual>
+        <collision>
+            <origin xyz="${chassis_length/2} 0 ${chassis_upper_height/2 + chassis_base_height + chassis_mid_height}"/>
+            <geometry>
+                <box size="${chassis_length} ${chassis_width} ${chassis_upper_height}"/>
+                <!-- <mesh filename="file://home/ros/ros/agv_ws/src/agv_ros/meshes/agv_body.stl"/> -->
+            </geometry>
+        </collision>
+        <xacro:inertial_box mass="${chassis_upper_mass}" x="${chassis_length}" y="${chassis_width}" z="${chassis_upper_height}">
+            <origin xyz="${chassis_length/2} 0 ${chassis_upper_height/2}" rpy="0 0 0"/>
+        </xacro:inertial_box>
+    </link>
+    <gazebo reference="upper_chassis">
         <material>Gazebo/White</material>
     </gazebo>

Commit message: Changing Robot Color

File: description/robot_core.xacro (robot description, xacro)
@@ -41,5 +41,5 @@
                 <box size="${chassis_length} ${chassis_width} ${chassis_base_height}"/>
             </geometry>
-            <material name="white"/>
+            <material name="orange"/>
         </visual>
         <collision>
@@ -54,5 +54,5 @@
     </link>
     <gazebo reference="chassis">
-        <material>Gazebo/White</material>
+        <material>Gazebo/Orange</material>
     </gazebo>
     <!-- MID CHASSIS LINK -->

Commit message: Adding Base Footprint

File: description/robot_core.xacro (robot description, xacro)
@@ -29,4 +29,11 @@
     <!-- BASE LINK -->
     <link name="base_link"></link>
+    <!-- BASE FOOTPRINT LINK -->
+    <joint name="base_footprint_joint" type="fixed">
+        <parent link="base_link"/>
+        <child link="base_footprint"/>
+        <origin xyz="0 0 0" rpy="0 0 0"/>
+    </joint>
+    <link name="base_footprint"></link>
     <!-- BASE CHASSIS LINK -->
     <joint name="chassis_joint" type="fixed">

Commit message: Tidying Up Files

File: description/robot_core.xacro (robot description, xacro)
@@ -6,5 +6,5 @@
     <!-- DEFINE ROBOT PROPERTIES -->
     <xacro:property name="chassis_length" value="0.650"/>
-    <xacro:property name="chassis_width" value="0.500"/>
+    <xacro:property name="chassis_width" value="0.600"/>
     <xacro:property name="chassis_height" value="0.320"/>
     <xacro:property name="chassis_base_height" value="0.052"/>
